Commit message: fix:调整sdk接口

File: lib/config/FastTouchV2.SLDASM.urdf (robot description, URDF)
Before this commit: robot FastTouchV2.SLDASM, 7 links, 6 joints
Links:
- link base_link: geometry collision mesh filename=./meshes/base_link.STL; visual mesh filename=./meshes/base_link.STL
- link link1: geometry collision mesh filename=./meshes/link1.STL; visual mesh filename=./meshes/link1.STL
- link link2: geometry collision mesh filename=./meshes/link2.STL; visual mesh filename=./meshes/link2.STL
- link link3: geometry collision mesh filename=./meshes/link3.STL; visual mesh filename=./meshes/link3.STL
- link link4: geometry collision mesh filename=./meshes/link4.STL; visual mesh filename=./meshes/link4.STL
- link link5: geometry collision mesh filename=./meshes/link5.STL; visual mesh filename=./meshes/link5.STL
- link link6: mass 0.8581 -> 0.5581; geometry collision mesh filename=./meshes/link6.STL; visual mesh filename=./meshes/link6.STL
Joints:
- joint joint4: limit lower=-1.710 upper=1.710 effort=7 velocity=20.9 -> lower=-1.710 upper=1.710 effort=12.5 velocity=20.9
