Commit message: fix:调整urdf和config

File: src/config/FastTouchV2.SLDASM.urdf (robot description, URDF)
Before this commit: robot FastTouchV2.SLDASM, 7 links, 6 joints
Joints:
- joint joint2: limit lower=-0.209 upper=3.508 effort=27 velocity=5.5 -> lower=-0.366 upper=3.508 effort=27 velocity=5.5

Commit message: 合并本地轨迹回放和配置修改

File: src/config/FastTouchV2.SLDASM.urdf (robot description, URDF)
Before this commit: robot FastTouchV2.SLDASM, 7 links, 6 joints
Joints:
- joint joint4: limit lower=-1.710 upper=1.710 effort=12.5 velocity=20.9 -> lower=-1.710 upper=1.710 effort=7 velocity=20.9
